File: cpLeoNode_V3_0.sch (EAGLE design)
At the start: 45 parts, among them CON6 0.100, CON7 0.100, J1 0.100, J2 0.100, P1 CA CC, U1 MAX3465CPD, U2 NE555P

Commit message: A bunch of cleanup after moving things around
1 - move Arduino connectors closer together for better fit with the Leonardo
2 - added VCC plane and removed a lot of old VCC and GND traces
3- added labels on top to help orient Leonardo
4 - mirrored bottom labels and moved to bplace for readability
Other:
- note added: "Rev: v3.3"
- note removed: "Rev: v3.1"
Changed lines of the file:
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@@
 <wire x1="162.56" y1="215.9" x2="124.46" y2="215.9" width="0.1524" layer="97"/>
 <wire x1="124.46" y1="215.9" x2="124.46" y2="193.04" width="0.1524" layer="97"/>
-<text x="279.4" y="2.54" size="1.27" layer="97" font="vector">Rev: v3.1</text>
+<text x="279.4" y="2.54" size="1.27" layer="97" font="vector">Rev: v3.3</text>
 <text x="248.92" y="1.27" size="1.27" layer="97" font="vector">Date: 03/04/2018
 08/20/19, 05/06/22</text>
